File: StringCar_M0_Express/StringCar_M0_Express.sch (KiCad schematic (older format))
At the start: 39 parts, among them J1 USB_MICRO, J2 SENSOR_IN, J3 SWD, J4 STEMMA-QT, J5 MOTOR, J6 LIPO_BATT, Q1 DMG2305UX-13, Q2 DMG2305UX-13, SW1 RESET, SW2 POWER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

Commit message: update pcb layout and logo graphics
Parts:
- removed F1: 0ZCG0050AF2C, Resistors_SMD:R_1812, symbol device:Polyfuse_Small
- added C8: 0.01uF, Capacitors_SMD:C_0805, symbol device:C_Small
- LED1, LED3: footprint Adafruit:D_0805_hand_soldering -> LEDs:LED_0805
Connections:
- net labels removed: Vsw
- wire segments 201 -> 204
Other:
- note removed: "30V / 0.5A"
Changed lines of the file:
@@
 Sheet 1 1
 Title "StringCar_M0_Express"
-Date "2019-10-02"
-Rev "v03"
+Date "2019-10-20"
+Rev "v04"
 Comp "Cedar Grove Studios"
 Comment1 ""
@@
 F 0 "LED1" V 11575 1350 50  0000 C CNN
 F 1 "RED" V 11475 1350 50  0000 C CNN
-F 2 "Adafruit:D_0805_hand_soldering" H 11475 1475 50  0001 C CNN
+F 2 "LEDs:LED_0805" H 11475 1475 50  0001 C CNN
 F 3 "" H 11475 1475 50  0001 C CNN
 	1    11475 1475
@@
 F 0 "LED3" V 2475 5700 50  0000 C CNN
 F 1 "ORG" V 2375 5700 50  0000 C CNN
-F 2 "Adafruit:D_0805_hand_soldering" H 2375 5825 50  0001 C CNN
+F 2 "LEDs:LED_0805" H 2375 5825 50  0001 C CNN
 F 3 "" H 2375 5825 50  0001 C CNN
 	1    2375 5825
@@
 U 1 1 5D0F3715
 P 6400 6900
-F 0 "C4" H 6200 6975 50  0000 L CNN
-F 1 "220uF" H 6075 6900 50  0000 L CNN
+F 0 "C4" H 6475 6975 50  0000 L CNN
+F 1 "220uF" H 6475 6900 50  0000 L CNN
 F 2 "Adafruit:CP_Elect_6.6x6.6" H 6400 6900 50  0001 C CNN
 F 3 "" H 6400 6900 50  0001 C CNN
@@
 	13050 1550 13050 1725
 $Comp
-L device:Polyfuse_Small F1
-U 1 1 5D90F1AE
-P 6050 6350
-F 0 "F1" V 6225 6350 50  0000 C CNN
-F 1 "0ZCG0050AF2C" V 6150 6350 50  0000 C CNN
-F 2 "Resistors_SMD:R_1812" H 6100 6150 50  0001 L CNN
-F 3 "" H 6050 6350 50  0001 C CNN
-	1    6050 6350
-	0    1    1    0
-$EndComp
-Wire Wire Line
-	6150 6350 6400 6350
-$Comp
 L dk_Transistors-FETs-MOSFETs-Single:DMG2305UX-13 Q1
 U 1 1 5D935606
@@
 U 1 1 5D941007
 P 4550 6875
-F 0 "R10" H 4450 6825 50  0000 C CNN
+F 0 "R10" H 4425 6825 50  0000 C CNN
 F 1 "100K" H 4300 6900 50  0000 L CNN
 F 2 "Resistors_SMD:R_0805" H 4550 6875 50  0001 C CNN
@@
 Wire Wire Line
 	4250 5800 4250 5450
-Wire Wire Line
-	5950 6350 5800 6350
 Wire Wire Line
 	6400 6500 6550 6500
@@
 Wire Wire Line
 	5100 5600 5100 5450
-Text Notes 5825 6625 0    50   ~ 0
-30V / 0.5A
 Wire Wire Line
 	1875 7300 2750 7300
-Text Label 5825 6350 0    50   ~ 0
-Vsw
 Text Label 4875 6350 0    50   ~ 0
 Vbus
@@
 Wire Wire Line
 	7850 3375 8575 3375
+$Comp
+L device:C_Small C8
+U 1 1 5DAE13E0
+P 6175 6900
+F 0 "C8" H 6000 6975 50  0000 L CNN
+F 1 "0.01uF" H 5850 6900 50  0000 L CNN
+F 2 "Capacitors_SMD:C_0805" H 6175 6900 50  0001 C CNN
+F 3 "" H 6175 6900 50  0001 C CNN
+	1    6175 6900
+	1    0    0    -1
+$EndComp
+Wire Wire Line
+	5800 6350 6175 6350
+Wire Wire Line
+	6400 7250 6175 7250
+Wire Wire Line
+	6175 7250 6175 7000
+Connection ~ 6400 7250
+Wire Wire Line
+	6175 6800 6175 6350
+Connection ~ 6175 6350
+Wire Wire Line
+	6175 6350 6400 6350
 $EndSCHEMATC

Commit message: update footprints
Other:
- note added: "2MB (16Mbit) Flash"
- note removed: "8MB (64Mbit) Flash"
Changed lines of the file:
@@
 Internal SPI on SERCOM2
 Text Notes 6900 2100 0    50   ~ 0
-8MB (64Mbit) Flash
+2MB (16Mbit) Flash
 Wire Wire Line
 	7200 1600 7750 1600

Commit message: repair schematic and regenerate PCB as v05
Changed lines of the file:
@@
 Sheet 1 1
 Title "StringCar_M0_Express"
-Date "2019-10-20"
-Rev "v04"
+Date "2020-01-18"
+Rev "v05"
 Comp "Cedar Grove Studios"
 Comment1 ""
@@
 U 1 1 5D24DA51
 P 5400 7050
-F 0 "SW2" V 5325 7300 50  0000 C CNN
-F 1 "POWER" V 5400 7350 50  0000 C CNN
+F 0 "SW2" V 5300 6875 50  0000 C CNN
+F 1 "POWER" V 5375 6825 50  0000 C CNN
 F 2 "Adafruit:SW_SPDT_CK-JS102011SAQN" H 5400 7050 50  0001 C CNN
 F 3 "" H 5400 7050 50  0001 C CNN
 	1    5400 7050
-	0    1    1    0
+	0    -1   1    0
 $EndComp
 Text Label 6400 5850 0    50   ~ 0
@@
 F 12 "Active" H 5300 7100 60  0001 L CNN "Status"
 	1    5100 5900
-	1    0    0    -1
+	1    0    0    1
 $EndComp
 $Comp
@@
 	4250 6350 4550 6350
 Wire Wire Line
-	4250 6350 4250 5800
+	4250 6350 4250 6000
 Connection ~ 4250 6350
 Wire Wire Line
-	4250 5800 4700 5800
-Connection ~ 4250 5800
-Wire Wire Line
-	4250 5800 4250 5450
+	4250 6000 4700 6000
 Wire Wire Line
 	6400 6500 6550 6500
@@
 Wire Wire Line
 	6175 6350 6400 6350
+Connection ~ 4250 6000
+Wire Wire Line
+	4250 5450 4250 6000
 $EndSCHEMATC

Commit message: update schematic with symbol correction; add warning
Other:
- note added: "WARNING: The stock schematic symbol for the\nDMG2305UX-13 provided by DigiKey incorrectly\nswapped source and drain. The corrected\nsymbol is shown here."
Changed lines of the file:
@@
 	1    0    0    -1
 $EndComp
-Text Notes 5775 7625 0    50   ~ 0
+Text Notes 6325 7750 0    50   ~ 0
 Power Management
 $Comp
@@
 Wire Wire Line
 	4250 5450 4250 6000
+Text Notes 3850 7925 0    50   ~ 0
+WARNING: The stock schematic symbol for the\nDMG2305UX-13 provided by DigiKey incorrectly\nswapped source and drain. The corrected\nsymbol is shown here.
 $EndSCHEMATC
