File: StringCar_M0_Express/StringCar_M0_Express.sch (KiCad schematic (older format))
At the start: 39 parts, among them J1 USB_MICRO, J2 SENSOR_IN, J3 SWD, J4 STEMMA-QT, J5 MOTOR, J6 LIPO_BATT, Q1 DMG2305UX-13, Q2 DMG2305UX-13, SW1 RESET, SW2 POWER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

Commit message: update schematic
Other:
- note added: "Consider a TPS2000CDGNR\npower switch/manager chip"
Changed lines of the file:
@@
 Text Notes 3850 7925 0    50   ~ 0
 WARNING: The stock schematic symbol for the\nDMG2305UX-13 provided by DigiKey incorrectly\nswapped source and drain. The corrected\nsymbol is shown here.
+Text Notes 6000 5675 0    100  ~ 0
+Consider a TPS2000CDGNR\npower switch/manager chip
 $EndSCHEMATC
